Commit message: adjusted joint names, updated configs

File: robot_specific_config/abb_irb1200_5_90_moveit_config/config/abb_irb1200_5_90_macro.srdf.xacro (robot description, xacro)
@@ -3,28 +3,50 @@
   <xacro:macro name="abb_irb1200_5_90_srdf">
     <group name="manipulator">
-        <chain base_link="base_link" tip_link="tool0" />
+        <chain base_link="base_link" tip_link="tool0"/>
+    </group>
+    <group name="extax">
+        <joint name="ext_joint_1"/>
+    </group>
+    <group name="whole_station">
+        <joint name="ext_joint_1"/>
+        <joint name="rob1_joint_1"/>
+        <joint name="rob1_joint_2"/>
+        <joint name="rob1_joint_3"/>
+        <joint name="rob1_joint_4"/>
+        <joint name="rob1_joint_5"/>
+        <joint name="rob1_joint_6"/>
     </group>
     <!--GROUP STATES: Purpose: Define a named state for a particular group, in terms of joint values. This is useful to define states like 'folded arms'-->
     <group_state name="all_zero" group="manipulator">
-        <joint name="joint_1" value="0" />
-        <joint name="joint_2" value="0" />
-        <joint name="joint_3" value="0" />
-        <joint name="joint_4" value="0" />
-        <joint name="joint_5" value="0" />
-        <joint name="joint_6" value="0" />
+        <joint name="rob1_joint_1" value="0"/>
+        <joint name="rob1_joint_2" value="0"/>
+        <joint name="rob1_joint_3" value="0"/>
+        <joint name="rob1_joint_4" value="0"/>
+        <joint name="rob1_joint_5" value="0"/>
+        <joint name="rob1_joint_6" value="-0.009"/>
+    </group_state>
+    <group_state name="zeros" group="extax">
+        <joint name="ext_joint_1" value="0"/>
     </group_state>
     <!--VIRTUAL JOINT: Purpose: this element defines a virtual joint between a robot link and an external frame of reference (considered fixed with respect to the robot)-->
     <virtual_joint type="floating" parent_frame="world" child_link="base_link" />
     <!--DISABLE COLLISIONS: By default it is assumed that any link of the robot could potentially come into collision with any other link in the robot. This tag disables collision checking between a specified pair of links. -->
-    <disable_collisions link1="base_link" link2="link_1" reason="Adjacent" />
-    <disable_collisions link1="link_1" link2="link_2" reason="Adjacent" />
-    <disable_collisions link1="link_2" link2="link_3" reason="Adjacent" />
-    <disable_collisions link1="link_2" link2="link_5" reason="Never" />
-    <disable_collisions link1="link_2" link2="link_6" reason="Never" />
-    <disable_collisions link1="link_3" link2="link_4" reason="Adjacent" />
-    <disable_collisions link1="link_3" link2="link_5" reason="Never" />
-    <disable_collisions link1="link_3" link2="link_6" reason="Never" />
-    <disable_collisions link1="link_4" link2="link_5" reason="Adjacent" />
-    <disable_collisions link1="link_5" link2="link_6" reason="Adjacent" />
+    <disable_collisions link1="base_link" link2="extax_link" reason="Adjacent"/>
+    <disable_collisions link1="base_link" link2="link_1" reason="Adjacent"/>
+    <disable_collisions link1="extax_link" link2="link_1" reason="Never"/>
+    <disable_collisions link1="extax_link" link2="link_2" reason="Never"/>
+    <disable_collisions link1="link_1" link2="link_2" reason="Adjacent"/>
+    <disable_collisions link1="link_1" link2="panels" reason="Never"/>
+    <disable_collisions link1="link_1" link2="table" reason="Never"/>
+    <disable_collisions link1="link_2" link2="link_3" reason="Adjacent"/>
+    <disable_collisions link1="link_2" link2="link_5" reason="Never"/>
+    <disable_collisions link1="link_2" link2="link_6" reason="Never"/>
+    <disable_collisions link1="link_3" link2="link_4" reason="Adjacent"/>
+    <disable_collisions link1="link_3" link2="link_5" reason="Never"/>
+    <disable_collisions link1="link_3" link2="link_6" reason="Never"/>
+    <disable_collisions link1="link_4" link2="link_5" reason="Adjacent"/>
+    <disable_collisions link1="link_5" link2="link_6" reason="Adjacent"/>
+    <disable_collisions link1="link_5" link2="toolFrame" reason="Never"/>
+    <disable_collisions link1="link_6" link2="toolFrame" reason="Adjacent"/>
   </xacro:macro>
 </robot>

File: robot_specific_config/abb_irb1200_support/urdf/irb1200.ros2_control.xacro (robot description, xacro)
@@ -16,11 +16,11 @@
           <param name="rws_ip">${rws_ip}</param>
           <!-- The following parameter is used for non-MultiMove only -->
-          <param name="egm_port">6511</param>
+          <!--param name="egm_port">6511</param-->
           <!-- The following parameters are used for the MultiMove example only -->
-          <!-- <param name="rob1egm_port">6511</param> -->
-          <!-- <param name="extaxegm_port">6512</param> -->
+          <param name="rob1egm_port">6511</param>
+          <param name="extaxegm_port">6512</param>
         </xacro:unless>
       </hardware>
-      <joint name="${prefix}joint_1">
+      <joint name="${prefix}rob1_joint_1">
         <command_interface name="position">
           <param name="min">{-2*pi}</param>
@@ -33,5 +33,5 @@
         <state_interface name="velocity"/>
       </joint>
-      <joint name="${prefix}joint_2">
+      <joint name="${prefix}rob1_joint_2">
         <command_interface name="position">
           <param name="min">-2.41</param>
@@ -44,5 +44,5 @@
         <state_interface name="velocity"/>
       </joint>
-      <joint name="${prefix}joint_3">
+      <joint name="${prefix}rob1_joint_3">
         <command_interface name="position">
           <param name="min">{-2*pi}</param>
@@ -55,5 +55,5 @@
         <state_interface name="velocity"/>
       </joint>
-      <joint name="${prefix}joint_4">
+      <joint name="${prefix}rob1_joint_4">
         <command_interface name="position">
           <param name="min">-2.66</param>
@@ -66,5 +66,5 @@
         <state_interface name="velocity"/>
       </joint>
-      <joint name="${prefix}joint_5">
+      <joint name="${prefix}rob1_joint_5">
         <command_interface name="position">
           <param name="min">{-2*pi}</param>
@@ -77,5 +77,5 @@
         <state_interface name="velocity"/>
       </joint>
-      <joint name="${prefix}joint_6">
+      <joint name="${prefix}rob1_joint_6">
         <command_interface name="position">
           <param name="min">-2.23</param>
@@ -88,4 +88,13 @@
         <state_interface name="velocity"/>
       </joint>
+      <joint name="${prefix}ext_joint_1">
+        <command_interface name="position">
+        </command_interface>
+        <command_interface name="velocity"/>
+        <state_interface name="position">
+          <param name="initial_value">0.0</param>
+        </state_interface>
+        <state_interface name="velocity"/>
+      </joint>
     </ros2_control>
   </xacro:macro>

File: robot_specific_config/abb_irb1200_support/urdf/irb1200_5_90_macro.xacro (robot description, xacro)
@@ -143,7 +143,31 @@
       </visual>
     </link>
+    <link name="${prefix}extax_link">
+      <inertial>
+        <mass value="0.137"/>
+        <origin xyz="0.6 0.150 0.0" rpy="0 0 0"/>
+        <inertia ixx="0.001" ixy="0" ixz="0" iyy="0.001" iyz="0" izz="0.001"/>
+      </inertial>
+      <!-- Meshlab calculated values (below) make gazebo crash when rotating this joint. -->
+      <!-- <inertial>
+        <mass value="0.00686711"/>
+        <origin xyz="-0.00250976 -1.89e-06 0.00010218"/>
+        <inertia ixx="1.3517e-06" ixy="-1.21316e-11" ixz="9.18065e-12" iyy="6.89813e-07" iyz="-1.21534e-10" izz="6.90097e-07"/>
+      </inertial> -->
+      <!--collision name="collision">
+        <geometry>
+          <mesh filename="package://abb_irb1200_support/meshes/irb1200_5_90/collision/link_6.stl"/>
+        </geometry>
+      </collision>
+      <visual name="visual">
+        <geometry>
+          <mesh filename="package://abb_irb1200_support/meshes/irb1200_5_90/visual/link_6.dae"/>
+        </geometry>
+        <xacro:material_abb_yellow />
+      </visual-->
+    </link>
     <!-- end of link list -->
     <!-- joint list -->
-    <joint type="revolute" name="${prefix}joint_1">
+    <joint type="revolute" name="${prefix}rob1_joint_1">
       <origin xyz="0 0 0.3991" rpy="0 0 0"/>
       <axis xyz="0 0 1"/>
@@ -154,5 +178,5 @@
       <dynamics damping="50.0" friction="1.0"/>
     </joint>
-    <joint type="revolute" name="${prefix}joint_2">
+    <joint type="revolute" name="${prefix}rob1_joint_2">
       <origin xyz="0 0 0" rpy="0 0 0"/>
       <axis xyz="0 1 0"/>
@@ -163,5 +187,5 @@
       <dynamics damping="50.0" friction="1.0"/>
     </joint>
-    <joint type="revolute" name="${prefix}joint_3">
+    <joint type="revolute" name="${prefix}rob1_joint_3">
       <origin xyz="0 0 0.448" rpy="0 0 0"/>
       <axis xyz="0 1 0"/>
@@ -172,5 +196,5 @@
       <dynamics damping="10.0" friction="1.0"/>
     </joint>
-    <joint type="revolute" name="${prefix}joint_4">
+    <joint type="revolute" name="${prefix}rob1_joint_4">
       <origin xyz="0 0 0.042" rpy="0 0 0"/>
       <axis xyz="1 0 0"/>
@@ -181,5 +205,5 @@
       <dynamics damping="5.0" friction="1.0"/>
     </joint>
-    <joint type="revolute" name="${prefix}joint_5">
+    <joint type="revolute" name="${prefix}rob1_joint_5">
       <origin xyz="0.451 0 0" rpy="0 0 0"/>
       <axis xyz="0 1 0"/>
@@ -190,5 +214,5 @@
       <dynamics damping="2.0" friction="1.0"/>
     </joint>
-    <joint type="revolute" name="${prefix}joint_6">
+    <joint type="revolute" name="${prefix}rob1_joint_6">
       <origin xyz="0.082 0 0" rpy="0 0 0"/>
       <axis xyz="1 0 0"/>
@@ -197,4 +221,12 @@
       <!-- See note 2 in package.xml about effort limits and dynamics values -->
       <limit effort="1000" lower="-6.283" upper="6.283" velocity="10.472"/>
+      <dynamics damping="1.0" friction="1.0"/>
+    </joint>
+    <joint type="continuous" name="${prefix}ext_joint_1">
+      <origin xyz="0.082 0 0" rpy="0 0 0"/>
+      <axis xyz="1 0 0"/>
+      <parent link="${prefix}base_link"/>
+      <child link="${prefix}extax_link"/>
+      <limit effort="1000" velocity="10.472"/>
       <dynamics damping="1.0" friction="1.0"/>
     </joint>

Commit message: Compiles against Humble
seems to work!

File: robot_specific_config/abb_irb1200_5_90_moveit_config/config/abb_irb1200_5_90_macro.srdf.xacro (robot description, xacro)
@@ -49,4 +49,9 @@
     <disable_collisions link1="link_5" link2="toolFrame" reason="Never"/>
     <disable_collisions link1="link_6" link2="toolFrame" reason="Adjacent"/>
+    <disable_collisions link1="base_link" link2="panels" reason="Adjacent"/>
+    <disable_collisions link1="base_link" link2="table" reason="Adjacent"/>
+    <disable_collisions link1="extax_link" link2="panels" reason="Never"/>
+    <disable_collisions link1="extax_link" link2="table" reason="Default"/>
+    <disable_collisions link1="panels" link2="table" reason="Default"/>
   </xacro:macro>
 </robot>

File: robot_specific_config/abb_irb1200_support/urdf/irb1200_5_90_macro.xacro (robot description, xacro)
@@ -4,4 +4,37 @@
   <xacro:macro name="abb_irb1200_5_90" params="prefix">
     <!-- link list -->
+    <link name="table">
+    <collision>
+      <origin rpy = "0 0 0" xyz="0 0 0"/>
+      <geometry>
+        <mesh filename="package://abb_irb1200_support/meshes/irb1200_5_90/scene/kb06_base_no_chuck.stl"/>
+      </geometry>
+    </collision>
+    <visual>
+      <origin rpy = "0 0 0" xyz="0 0 0"/>
+      <geometry>
+        <mesh filename="package://abb_irb1200_support/meshes/irb1200_5_90/scene/kb06_base_no_chuck.stl"/>
+      </geometry>
+      <xacro:material_abb_pebble_gray />
+    </visual>
+  </link>
+  <link name="panels">
+    <collision name="collision">
+      <origin rpy = "0 0 0" xyz="0 0 0"/>
+        <geometry>
+          <mesh filename="package://abb_irb1200_support/meshes/irb1200_5_90/scene/panels_oversized.stl"/>
+      </geometry>
+    </collision>
+    <visual>
+      <origin rpy = "0 0 0" xyz="0 0 0"/>
+      <geometry>
+        <mesh filename="package://abb_irb1200_support/meshes/irb1200_5_90/scene/panels_oversized.stl"/>
+      </geometry>
+      <material name="">
+        <color rgba="0 0 0 0"/>
+      </material>
+      <!--xacro:material_abb_clear /-->
+    </visual>
+  </link>
     <link name="${prefix}base_link">
       <!-- See note 1 in package.xml about the inertial and mass values -->
@@ -149,4 +182,17 @@
         <inertia ixx="0.001" ixy="0" ixz="0" iyy="0.001" iyz="0" izz="0.001"/>
       </inertial>
+        <collision>
+          <origin rpy = "0 0 0" xyz="0 0 0"/>
+          <geometry>
+            <mesh filename="package://abb_irb1200_support/meshes/irb1200_5_90/scene/3RChuckAsm.stl"/>
+          </geometry>
+        </collision>
+        <visual>
+          <origin rpy = "0 0 0" xyz="0 0 0"/>
+          <geometry>
+            <mesh filename="package://abb_irb1200_support/meshes/irb1200_5_90/scene/3RChuckAsm.stl"/>
+          </geometry>
+          <xacro:material_abb_pebble_gray />
+        </visual>
       <!-- Meshlab calculated values (below) make gazebo crash when rotating this joint. -->
       <!-- <inertial>
@@ -224,6 +270,6 @@
     </joint>
     <joint type="continuous" name="${prefix}ext_joint_1">
-      <origin xyz="0.082 0 0" rpy="0 0 0"/>
-      <axis xyz="1 0 0"/>
+      <origin xyz="0.6096 0 0.100838" rpy="0 0 0"/>
+      <axis xyz="0 0 1"/>
       <parent link="${prefix}base_link"/>
       <child link="${prefix}extax_link"/>
@@ -253,4 +299,14 @@
       <child link="${prefix}tool0" />
     </joint>
+    <joint name="${prefix}base_link-table" type="fixed">
+      <origin xyz="0 0 0" rpy="0 0 0"/>
+      <parent link="${prefix}base_link"/>
+      <child link="${prefix}table"/>
+    </joint>
+    <joint name="${prefix}base_link-panels" type="fixed">
+      <origin xyz="0 0 0" rpy="0 0 0"/>
+      <parent link="${prefix}base_link"/>
+      <child link="${prefix}panels"/>
+    </joint>
   </xacro:macro>
 </robot>
