Commit message: Currently working kind of.

File: robot_specific_config/abb_irb1200_5_90_moveit_config/config/abb_irb1200_5_90_macro.srdf.xacro (robot description, xacro)
@@ -1,57 +1,68 @@
 <?xml version="1.0" encoding="utf-8"?>
 <robot xmlns:xacro="http://wiki.ros.org/xacro">
-  <xacro:macro name="abb_irb1200_5_90_srdf">
-    <group name="manipulator">
-        <chain base_link="base_link" tip_link="tool0"/>
-    </group>
-    <group name="extax">
-        <joint name="ext_joint_1"/>
-    </group>
-    <group name="whole_station">
-        <joint name="ext_joint_1"/>
-        <joint name="rob1_joint_1"/>
-        <joint name="rob1_joint_2"/>
-        <joint name="rob1_joint_3"/>
-        <joint name="rob1_joint_4"/>
-        <joint name="rob1_joint_5"/>
-        <joint name="rob1_joint_6"/>
-    </group>
-    <!--GROUP STATES: Purpose: Define a named state for a particular group, in terms of joint values. This is useful to define states like 'folded arms'-->
-    <group_state name="all_zero" group="manipulator">
-        <joint name="rob1_joint_1" value="0"/>
-        <joint name="rob1_joint_2" value="0"/>
-        <joint name="rob1_joint_3" value="0"/>
-        <joint name="rob1_joint_4" value="0"/>
-        <joint name="rob1_joint_5" value="0"/>
-        <joint name="rob1_joint_6" value="-0.009"/>
-    </group_state>
-    <group_state name="zeros" group="extax">
-        <joint name="ext_joint_1" value="0"/>
-    </group_state>
-    <!--VIRTUAL JOINT: Purpose: this element defines a virtual joint between a robot link and an external frame of reference (considered fixed with respect to the robot)-->
-    <virtual_joint type="floating" parent_frame="world" child_link="base_link" />
-    <!--DISABLE COLLISIONS: By default it is assumed that any link of the robot could potentially come into collision with any other link in the robot. This tag disables collision checking between a specified pair of links. -->
-    <disable_collisions link1="base_link" link2="extax_link" reason="Adjacent"/>
-    <disable_collisions link1="base_link" link2="link_1" reason="Adjacent"/>
-    <disable_collisions link1="extax_link" link2="link_1" reason="Never"/>
-    <disable_collisions link1="extax_link" link2="link_2" reason="Never"/>
-    <disable_collisions link1="link_1" link2="link_2" reason="Adjacent"/>
-    <disable_collisions link1="link_1" link2="panels" reason="Never"/>
-    <disable_collisions link1="link_1" link2="table" reason="Never"/>
-    <disable_collisions link1="link_2" link2="link_3" reason="Adjacent"/>
-    <disable_collisions link1="link_2" link2="link_5" reason="Never"/>
-    <disable_collisions link1="link_2" link2="link_6" reason="Never"/>
-    <disable_collisions link1="link_3" link2="link_4" reason="Adjacent"/>
-    <disable_collisions link1="link_3" link2="link_5" reason="Never"/>
-    <disable_collisions link1="link_3" link2="link_6" reason="Never"/>
-    <disable_collisions link1="link_4" link2="link_5" reason="Adjacent"/>
-    <disable_collisions link1="link_5" link2="link_6" reason="Adjacent"/>
-    <disable_collisions link1="link_5" link2="toolFrame" reason="Never"/>
-    <disable_collisions link1="link_6" link2="toolFrame" reason="Adjacent"/>
-    <disable_collisions link1="base_link" link2="panels" reason="Adjacent"/>
-    <disable_collisions link1="base_link" link2="table" reason="Adjacent"/>
-    <disable_collisions link1="extax_link" link2="panels" reason="Never"/>
-    <disable_collisions link1="extax_link" link2="table" reason="Default"/>
-    <disable_collisions link1="panels" link2="table" reason="Default"/>
-  </xacro:macro>
+    <xacro:macro name="abb_irb1200_5_90_srdf">
+        <group name="manipulator">
+            <chain base_link="base_link" tip_link="tool0"/>
+        </group>
+        <group name="extax">
+            <joint name="ext_joint_1"/>
+        </group>
+        <group name="whole_station">
+            <joint name="ext_joint_1"/>
+            <joint name="rob1_joint_1"/>
+            <joint name="rob1_joint_2"/>
+            <joint name="rob1_joint_3"/>
+            <joint name="rob1_joint_4"/>
+            <joint name="rob1_joint_5"/>            <joint name="rob1_joint_3" value="0.44897"/>
+            <joint name="rob1_joint_4" value="0.5662"/>
+            <joint name="rob1_joint_5" value="-0.67863"/>
+            <joint name="rob1_joint_6" value="-0.43109"/>
+            <joint name="rob1_joint_6"/>
+        </group>
+        <!--GROUP STATES: Purpose: Define a named state for a particular group, in terms of joint values. This is useful to define states like 'folded arms'-->
+        <group_state name="all_zero" group="manipulator">
+            <joint name="rob1_joint_1" value="0"/>
+            <joint name="rob1_joint_2" value="0"/>
+            <joint name="rob1_joint_3" value="0"/>
+            <joint name="rob1_joint_4" value="0"/>
+            <joint name="rob1_joint_5" value="0"/>
+            <joint name="rob1_joint_6" value="-0.009"/>
+        </group_state>
+        <group_state name="home" group="manipulator">
+            <joint name="rob1_joint_1" value="0.3895"/>
+            <joint name="rob1_joint_2" value="0.2527"/>
+            <joint name="rob1_joint_3" value="0.44897"/>
+            <joint name="rob1_joint_4" value="0.5662"/>
+            <joint name="rob1_joint_5" value="-0.67863"/>
+            <joint name="rob1_joint_6" value="-0.43109"/>
+        </group_state>
+        <group_state name="zeros" group="extax">
+            <joint name="ext_joint_1" value="0"/>
+        </group_state>
+        <!--VIRTUAL JOINT: Purpose: this element defines a virtual joint between a robot link and an external frame of reference (considered fixed with respect to the robot)-->
+        <virtual_joint type="floating" parent_frame="world" child_link="base_link"/>
+        <!--DISABLE COLLISIONS: By default it is assumed that any link of the robot could potentially come into collision with any other link in the robot. This tag disables collision checking between a specified pair of links. -->
+<!--        <disable_collisions link1="base_link" link2="extax_link" reason="Adjacent"/>-->
+        <disable_collisions link1="base_link" link2="link_1" reason="Adjacent"/>
+<!--        <disable_collisions link1="extax_link" link2="link_1" reason="Never"/>-->
+<!--        <disable_collisions link1="extax_link" link2="link_2" reason="Never"/>-->
+        <disable_collisions link1="link_1" link2="link_2" reason="Adjacent"/>
+<!--        <disable_collisions link1="link_1" link2="panels" reason="Never"/>-->
+        <disable_collisions link1="link_1" link2="table" reason="Never"/>
+        <disable_collisions link1="link_2" link2="link_3" reason="Adjacent"/>
+        <disable_collisions link1="link_2" link2="link_5" reason="Never"/>
+        <disable_collisions link1="link_2" link2="link_6" reason="Never"/>
+        <disable_collisions link1="link_3" link2="link_4" reason="Adjacent"/>
+        <disable_collisions link1="link_3" link2="link_5" reason="Never"/>
+        <disable_collisions link1="link_3" link2="link_6" reason="Never"/>
+        <disable_collisions link1="link_4" link2="link_5" reason="Adjacent"/>
+        <disable_collisions link1="link_5" link2="link_6" reason="Adjacent"/>
+        <disable_collisions link1="link_5" link2="toolFrame" reason="Never"/>
+        <disable_collisions link1="link_6" link2="toolFrame" reason="Adjacent"/>
+<!--        <disable_collisions link1="base_link" link2="panels" reason="Adjacent"/>-->
+        <disable_collisions link1="base_link" link2="table" reason="Adjacent"/>
+<!--        <disable_collisions link1="extax_link" link2="panels" reason="Never"/>-->
+<!--        <disable_collisions link1="extax_link" link2="table" reason="Default"/>-->
+<!--        <disable_collisions link1="panels" link2="table" reason="Default"/>-->
+    </xacro:macro>
 </robot>

File: robot_specific_config/abb_irb1200_support/urdf/irb1200.ros2_control.xacro (robot description, xacro)
@@ -1,101 +1,92 @@
 <?xml version="1.0"?>
 <robot xmlns:xacro="http://www.ros.org/wiki/xacro">
-  <xacro:macro name="abb_ros2_control" params="name prefix use_fake_hardware:=true rws_ip rws_port">
-    <ros2_control name="${name}" type="system">
-      <hardware>
-        <!-- ros2_control simulation -->
-        <xacro:if value="${use_fake_hardware}">
-          <plugin>fake_components/GenericSystem</plugin>
-          <param name="fake_sensor_commands">false</param>
-          <param name="state_following_offset">0.0</param>
-        </xacro:if>
-        <!-- physical hardware or RobotStudio simulation -->
-        <xacro:unless value="${use_fake_hardware}">
-          <plugin>abb_hardware_interface/ABBSystemPositionOnlyHardware</plugin>
-          <param name="rws_port">${rws_port}</param>
-          <param name="rws_ip">${rws_ip}</param>
-          <!-- The following parameter is used for non-MultiMove only -->
-          <!--param name="egm_port">6511</param-->
-          <!-- The following parameters are used for the MultiMove example only -->
-          <param name="rob1egm_port">6511</param>
-          <param name="extaxegm_port">6512</param>
-        </xacro:unless>
-      </hardware>
-      <joint name="${prefix}rob1_joint_1">
-        <command_interface name="position">
-          <param name="min">{-2*pi}</param>
-          <param name="max">{2*pi}</param>
-        </command_interface>
-        <command_interface name="velocity"/>
-        <state_interface name="position">
-          <param name="initial_value">0.0</param>
-        </state_interface>
-        <state_interface name="velocity"/>
-      </joint>
-      <joint name="${prefix}rob1_joint_2">
-        <command_interface name="position">
-          <param name="min">-2.41</param>
-          <param name="max">2.41</param>
-        </command_interface>
-        <command_interface name="velocity"/>
-        <state_interface name="position">
-          <param name="initial_value">0.0</param>
-        </state_interface>
-        <state_interface name="velocity"/>
-      </joint>
-      <joint name="${prefix}rob1_joint_3">
-        <command_interface name="position">
-          <param name="min">{-2*pi}</param>
-          <param name="max">{2*pi}</param>
-        </command_interface>
-        <command_interface name="velocity"/>
-        <state_interface name="position">
-          <param name="initial_value">0.0</param>
-        </state_interface>
-        <state_interface name="velocity"/>
-      </joint>
-      <joint name="${prefix}rob1_joint_4">
-        <command_interface name="position">
-          <param name="min">-2.66</param>
-          <param name="max">2.66</param>
-        </command_interface>
-        <command_interface name="velocity"/>
-        <state_interface name="position">
-          <param name="initial_value">0.0</param>
-        </state_interface>
-        <state_interface name="velocity"/>
-      </joint>
-      <joint name="${prefix}rob1_joint_5">
-        <command_interface name="position">
-          <param name="min">{-2*pi}</param>
-          <param name="max">{2*pi}</param>
-        </command_interface>
-        <command_interface name="velocity"/>
-        <state_interface name="position">
-          <param name="initial_value">0.0</param>
-        </state_interface>
-        <state_interface name="velocity"/>
-      </joint>
-      <joint name="${prefix}rob1_joint_6">
-        <command_interface name="position">
-          <param name="min">-2.23</param>
-          <param name="max">2.23</param>
-        </command_interface>
-        <command_interface name="velocity"/>
-        <state_interface name="position">
-          <param name="initial_value">0.0</param>
-        </state_interface>
-        <state_interface name="velocity"/>
-      </joint>
-      <joint name="${prefix}ext_joint_1">
-        <command_interface name="position">
-        </command_interface>
-        <command_interface name="velocity"/>
-        <state_interface name="position">
-          <param name="initial_value">0.0</param>
-        </state_interface>
-        <state_interface name="velocity"/>
-      </joint>
-    </ros2_control>
-  </xacro:macro>
+    <xacro:macro name="abb_ros2_control" params="name prefix use_fake_hardware:=true rws_ip rws_port">
+        <ros2_control name="${name}" type="system">
+            <hardware>
+                <!-- ros2_control simulation -->
+                <xacro:if value="${use_fake_hardware}">
+                    <plugin>fake_components/GenericSystem</plugin>
+                    <param name="fake_sensor_commands">false</param>
+                    <param name="state_following_offset">0.0</param>
+                </xacro:if>
+                <!-- physical hardware or RobotStudio simulation -->
+                <xacro:unless value="${use_fake_hardware}">
+                    <plugin>abb_hardware_interface/ABBSystemPositionOnlyHardware</plugin>
+                    <param name="rws_port">${rws_port}</param>
+                    <param name="rws_ip">${rws_ip}</param>
+                    <!-- The following parameter is used for non-MultiMove only -->
+                    <!--param name="egm_port">6511</param-->
+                    <!-- The following parameters are used for the MultiMove example only -->
+                    <param name="rob1egm_port">6511</param>
+                    <param name="extaxegm_port">6512</param>
+                </xacro:unless>
+            </hardware>
+            <joint name="${prefix}rob1_joint_1">
+                <command_interface name="position">
+                    <param name="min">{-2*pi}</param>
+                    <param name="max">{2*pi}</param>
+                </command_interface>
+                <command_interface name="velocity"/>
+                <state_interface name="position">
+                    <param name="initial_value">0.0</param>
+                </state_interface>
+                <state_interface name="velocity"/>
+            </joint>
+            <joint name="${prefix}rob1_joint_2">
+                <command_interface name="position">
+                    <param name="min">-2.41</param>
+                    <param name="max">2.41</param>
+                </command_interface>
+                <command_interface name="velocity"/>
+                <state_interface name="position">
+                    <param name="initial_value">0.0</param>
+                </state_interface>
+                <state_interface name="velocity"/>
+            </joint>
+            <joint name="${prefix}rob1_joint_3">
+                <command_interface name="position">
+                    <param name="min">{-2*pi}</param>
+                    <param name="max">{2*pi}</param>
+                </command_interface>
+                <command_interface name="velocity"/>
+                <state_interface name="position">
+                    <param name="initial_value">0.0</param>
+                </state_interface>
+                <state_interface name="velocity"/>
+            </joint>
+            <joint name="${prefix}rob1_joint_4">
+                <command_interface name="position">
+                    <param name="min">-2.66</param>
+                    <param name="max">2.66</param>
+                </command_interface>
+                <command_interface name="velocity"/>
+                <state_interface name="position">
+                    <param name="initial_value">0.0</param>
+                </state_interface>
+                <state_interface name="velocity"/>
+            </joint>
+            <joint name="${prefix}rob1_joint_5">
+                <command_interface name="position">
+                    <param name="min">{-2*pi}</param>
+                    <param name="max">{2*pi}</param>
+                </command_interface>
+                <command_interface name="velocity"/>
+                <state_interface name="position">
+                    <param name="initial_value">0.0</param>
+                </state_interface>
+                <state_interface name="velocity"/>
+            </joint>
+            <joint name="${prefix}rob1_joint_6">
+                <command_interface name="position">
+                    <param name="min">-2.23</param>
+                    <param name="max">2.23</param>
+                </command_interface>
+                <command_interface name="velocity"/>
+                <state_interface name="position">
+                    <param name="initial_value">0.0</param>
+                </state_interface>
+                <state_interface name="velocity"/>
+            </joint>
+        </ros2_control>
+    </xacro:macro>
 </robot>

File: robot_specific_config/abb_irb1200_support/urdf/irb1200_5_90.xacro (robot description, xacro)
@@ -7,10 +7,10 @@
         <xacro:arg name="rws_port" default="80"/>
         <xacro:property name="rws_port" value="$(arg rws_port)"/>
-<!--        <xacro:arg name="robot" default=""/>-->
-<!--        <xacro:property name="robot" value="$(arg robot)"/>-->
-        <!-- Robot description -->
+        <xacro:arg name="robot" default=""/>
+        <xacro:property name="robot" value="$(arg robot)"/>
+<!--         Robot description-->
         <xacro:include filename="$(find abb_irb1200_support)/urdf/irb1200_5_90_macro.xacro"/>
-<!--        <xacro:abb_irb1200_5_90 prefix="" robot="${robot}"/>-->
-        <xacro:abb_irb1200_5_90 prefix=""/>
+        <xacro:abb_irb1200_5_90 prefix="" robot="${robot}"/>
+<!--        <xacro:abb_irb1200_5_90 prefix=""/>-->
         <!-- ros2_control -->
         <xacro:include filename="$(find abb_irb1200_support)/urdf/irb1200.ros2_control.xacro"/>

File: robot_specific_config/abb_irb1200_support/urdf/irb1200_5_90_macro.xacro (robot description, xacro)
@@ -4,66 +4,14 @@
     <xacro:include filename="kb06_macro.xacro"/>
     <xacro:include filename="kb04-5_macro.xacro"/>
-    <xacro:macro name="abb_irb1200_5_90" params="prefix">
-<!--    <xacro:macro name="abb_irb1200_5_90" params="prefix robot">-->
-<!--        <xacro:property name="robot_property" value="${robot}"/>-->
-<!--        <xacro:if value="${robot_property == 'kb06'}">-->
-<!--            <xacro:kb06 prefix="${prefix}"/>-->
-<!--        </xacro:if>-->
-<!--        <xacro:if value="${robot_property == 'kb04'}">-->
-<!--            <xacro:kb04/>-->
-<!--        </xacro:if>-->
-        <link name="table">
-            <collision>
-                <origin rpy="0 0 0" xyz="0 0 0"/>
-                <geometry>
-                    <mesh filename="package://abb_irb1200_support/meshes/irb1200_5_90/scene/kb06_base_no_chuck.stl"/>
-                </geometry>
-            </collision>
-            <visual>
-                <origin rpy="0 0 0" xyz="0 0 0"/>
-                <geometry>
-                    <mesh filename="package://abb_irb1200_support/meshes/irb1200_5_90/scene/kb06_base_no_chuck.stl"/>
-                </geometry>
-                <xacro:material_abb_leaf_green/>
-            </visual>
-        </link>
-        <link name="panels">
-            <collision name="collision">
-                <origin rpy="0 0 0" xyz="0 0 0"/>
-                <geometry>
-                    <mesh filename="package://abb_irb1200_support/meshes/irb1200_5_90/scene/panels_oversized.stl"/>
-                </geometry>
-            </collision>
-            <visual>
-                <origin rpy="0 0 0" xyz="0 0 0"/>
-                <geometry>
-                    <mesh filename="package://abb_irb1200_support/meshes/irb1200_5_90/scene/panels_oversized.stl"/>
-                </geometry>
-                <material name="">
-                    <color rgba="0.5 0.5 0.5 0.2"/>
-                </material>
-                <!--xacro:material_abb_clear /-->
-            </visual>
-        </link>
-        <link name="${prefix}extax_link">
-            <inertial>
-                <mass value="0.137"/>
-                <origin xyz="0.6 0.150 0.0" rpy="0 0 0"/>
-                <inertia ixx="0.001" ixy="0" ixz="0" iyy="0.001" iyz="0" izz="0.001"/>
-            </inertial>
-            <collision>
-                <origin rpy="0 0 0" xyz="0 0 0"/>
-                <geometry>
-                    <mesh filename="package://abb_irb1200_support/meshes/irb1200_5_90/scene/3RChuckAsm.stl"/>
-                </geometry>
-            </collision>
-            <visual>
-                <origin rpy="0 0 0" xyz="0 0 0"/>
-                <geometry>
-                    <mesh filename="package://abb_irb1200_support/meshes/irb1200_5_90/scene/3RChuckAsm.stl"/>
-                </geometry>
-                <xacro:material_abb_pebble_gray/>
-            </visual>
-        </link>
+<!--    <xacro:macro name="abb_irb1200_5_90" params="prefix">-->
+    <xacro:macro name="abb_irb1200_5_90" params="prefix robot">
+        <!-- Check which robot is being used and load in appropriate xacro file -->
+        <xacro:property name="robot_property" value="${robot}"/>
+        <xacro:if value="${robot_property == 'kb06'}">
+            <xacro:kb06 prefix="${prefix}"/>
+        </xacro:if>
+        <xacro:if value="${robot_property == 'kb04'}">
+            <xacro:kb04 prefix="${prefix}"/>
+        </xacro:if>
         <link name="${prefix}base_link">
             <!-- See note 1 in package.xml about the inertial and mass values -->
@@ -264,12 +212,4 @@
             <!-- See note 2 in package.xml about effort limits and dynamics values -->
             <limit effort="1000" lower="-6.283" upper="6.283" velocity="10.472"/>
-            <dynamics damping="1.0" friction="1.0"/>
-        </joint>
-        <joint type="continuous" name="${prefix}ext_joint_1">
-            <origin xyz="0.6096 0 0.100838" rpy="0 0 0"/>
-            <axis xyz="0 0 1"/>
-            <parent link="${prefix}base_link"/>
-            <child link="${prefix}extax_link"/>
-            <limit effort="1000" velocity="10.472"/>
             <dynamics damping="1.0" friction="1.0"/>
         </joint>
@@ -296,14 +236,4 @@
             <child link="${prefix}tool0"/>
         </joint>
-        <joint name="${prefix}base_link-table" type="fixed">
-            <origin xyz="0 0 0" rpy="0 0 0"/>
-            <parent link="${prefix}base_link"/>
-            <child link="${prefix}table"/>
-        </joint>
-        <joint name="${prefix}base_link-panels" type="fixed">
-            <origin xyz="0 0 0" rpy="0 0 0"/>
-            <parent link="${prefix}base_link"/>
-            <child link="${prefix}panels"/>
-        </joint>
     </xacro:macro>
 </robot>
