Commit message: Currently working kind of.

File: robot_specific_config/abb_irb1200_support/urdf/kb04-5_macro.xacro (robot description, xacro)
@@ -1,5 +1,5 @@
 <?xml version="1.0"?>
 <robot xmlns:xacro="http://ros.org/wiki/xacro">
-    <xacro:macro  name="kb04">
+    <xacro:macro  name="kb04" params="prefix">
         <link name="table">
             <collision>
@@ -14,7 +14,24 @@
                     <mesh filename="package://abb_irb1200_support/meshes/irb1200_5_90/scene/kb04_Base_v3.stl"/>
                 </geometry>
-                <xacro:material_abb_pebble_gray/>
+                <xacro:material_abb_ultramarine_blue/>
             </visual>
         </link>
+        <joint name="${prefix}base_link-table" type="fixed">
+            <origin xyz="0.1459 0.2021 0" rpy="0 0 0"/>
+            <parent link="${prefix}base_link"/>
+            <child link="${prefix}table"/>
+        </joint>
+        <link name="${prefix}chuck"/>
+        <joint name="${prefix}base_link-chuck" type="fixed">
+            <origin xyz="0.756632 0.200927 0.102209" rpy="0.0001095 -0.0036872 -1.5748606"/>
+            <parent link="${prefix}base_link"/>
+            <child link="${prefix}chuck"/>
+        </joint>
+        <link name="${prefix}toolFrame"/>
+        <joint name="${prefix}base_link-toolFrame" type="fixed">
+            <origin xyz="0.0809969 0.0005848 0.219497" rpy="1.5726663 0.006046 -1.5707967"/>
+            <parent link="${prefix}tool0"/>
+            <child link="${prefix}toolFrame"/>
+        </joint>
     </xacro:macro>
 </robot>

File: robot_specific_config/abb_irb1200_support/urdf/kb06_macro.xacro (robot description, xacro)
@@ -55,4 +55,31 @@
             </visual>
         </link>
+        <joint name="${prefix}base_link-table" type="fixed">
+            <origin xyz="0 0 0" rpy="0 0 0"/>
+            <parent link="${prefix}base_link"/>
+            <child link="${prefix}table"/>
+        </joint>
+        <joint name="${prefix}base_link-panels" type="fixed">
+            <origin xyz="0 0 0" rpy="0 0 0"/>
+            <parent link="${prefix}base_link"/>
+            <child link="${prefix}panels"/>
+        </joint>
+        <joint type="continuous" name="${prefix}ext_joint_1">
+            <origin xyz="0.6096 0 0.100838" rpy="0 0 0"/>
+            <axis xyz="0 0 1"/>
+            <parent link="${prefix}base_link"/>
+            <child link="${prefix}extax_link"/>
+            <limit effort="1000" velocity="10.472"/>
+            <dynamics damping="1.0" friction="1.0"/>
+        </joint>
+        <joint name="${prefix}ext_joint_1">
+            <command_interface name="position">
+            </command_interface>
+            <command_interface name="velocity"/>
+            <state_interface name="position">
+                <param name="initial_value">0.0</param>
+            </state_interface>
+            <state_interface name="velocity"/>
+        </joint>
     </xacro:macro>
 </robot>

Commit message: changed home values

File: robot_specific_config/abb_irb1200_5_90_moveit_config/config/abb_irb1200_5_90_macro.srdf.xacro (robot description, xacro)
@@ -30,10 +30,10 @@
         </group_state>
         <group_state name="home" group="manipulator">
-            <joint name="rob1_joint_1" value="0.3895"/>
-            <joint name="rob1_joint_2" value="0.2527"/>
-            <joint name="rob1_joint_3" value="0.44897"/>
-            <joint name="rob1_joint_4" value="0.5662"/>
-            <joint name="rob1_joint_5" value="-0.67863"/>
-            <joint name="rob1_joint_6" value="-0.43109"/>
+            <joint name="rob1_joint_1" value="0.42577928960737016"/>
+            <joint name="rob1_joint_2" value="0.21565327380088078"/>
+            <joint name="rob1_joint_3" value="0.3686193877257924"/>
+            <joint name="rob1_joint_4" value="0.6880622135409175"/>
+            <joint name="rob1_joint_5" value="-0.7080416122464187"/>
+            <joint name="rob1_joint_6" value="-0.5671417005127892"/>
         </group_state>
         <group_state name="zeros" group="extax">

Commit message: Removed extax errors when using robot model loader

File: robot_specific_config/abb_irb1200_5_90_moveit_config/config/abb_irb1200_5_90_macro.srdf.xacro (robot description, xacro)
@@ -5,9 +5,9 @@
             <chain base_link="base_link" tip_link="tool0"/>
         </group>
-        <group name="extax">
-            <joint name="ext_joint_1"/>
-        </group>
+<!--        <group name="extax">-->
+<!--            <joint name="ext_joint_1"/>-->
+<!--        </group>-->
         <group name="whole_station">
-            <joint name="ext_joint_1"/>
+<!--            <joint name="ext_joint_1"/>-->
             <joint name="rob1_joint_1"/>
             <joint name="rob1_joint_2"/>
@@ -37,9 +37,9 @@
             <joint name="rob1_joint_6" value="-0.5671417005127892"/>
         </group_state>
-        <group_state name="zeros" group="extax">
-            <joint name="ext_joint_1" value="0"/>
-        </group_state>
+<!--        <group_state name="zeros" group="extax">-->
+<!--            <joint name="ext_joint_1" value="0"/>-->
+<!--        </group_state>-->
         <!--VIRTUAL JOINT: Purpose: this element defines a virtual joint between a robot link and an external frame of reference (considered fixed with respect to the robot)-->
-        <virtual_joint type="floating" parent_frame="world" child_link="base_link"/>
+        <virtual_joint name="world_link" type="floating" parent_frame="world" child_link="base_link"/>
         <!--DISABLE COLLISIONS: By default it is assumed that any link of the robot could potentially come into collision with any other link in the robot. This tag disables collision checking between a specified pair of links. -->
 <!--        <disable_collisions link1="base_link" link2="extax_link" reason="Adjacent"/>-->

File: robot_specific_config/abb_irb1200_support/urdf/irb1200.ros2_control.xacro (robot description, xacro)
@@ -16,8 +16,8 @@
                     <param name="rws_ip">${rws_ip}</param>
                     <!-- The following parameter is used for non-MultiMove only -->
-                    <param name="egm_port">6511</param>
+<!--                    <param name="egm_port">6511</param>-->
                     <!-- The following parameters are used for the MultiMove example only -->
-                    <!--param name="rob1egm_port">6511</param>
-                    <param name="extaxegm_port">6512</param-->
+                    <param name="rob1egm_port">6511</param>
+                    <param name="extaxegm_port">6512</param>
                 </xacro:unless>
             </hardware>
