Commit message: not working

File: robot_specific_config/abb_irb1200_5_90_moveit_config/config/abb_irb1200_5_90.srdf.xacro (robot description, xacro)
@@ -1,5 +1,7 @@
 <?xml version="1.0" encoding="utf-8"?>
 <robot xmlns:xacro="http://wiki.ros.org/xacro" name="abb_irb1200_5_90">
+  <xacro:arg name="use_extax" default="None"/>
+  <xacro:property name="use_extax" value="$(arg use_extax)"/>
   <xacro:include filename="$(find abb_irb1200_5_90_moveit_config)/config/abb_irb1200_5_90_macro.srdf.xacro"/>
-  <xacro:abb_irb1200_5_90_srdf/>
+  <xacro:abb_irb1200_5_90_srdf use_extax="${use_extax}"/>
 </robot>

File: robot_specific_config/abb_irb1200_5_90_moveit_config/config/abb_irb1200_5_90_macro.srdf.xacro (robot description, xacro)
@@ -1,23 +1,11 @@
 <?xml version="1.0" encoding="utf-8"?>
 <robot xmlns:xacro="http://wiki.ros.org/xacro">
-    <xacro:macro name="abb_irb1200_5_90_srdf">
+    <xacro:macro name="abb_irb1200_5_90_srdf" params="use_extax">
         <group name="manipulator">
             <chain base_link="base_link" tip_link="tool0"/>
         </group>
-<!--        <group name="extax">-->
-<!--            <joint name="ext_joint_1"/>-->
-<!--        </group>-->
-        <group name="whole_station">
-<!--            <joint name="ext_joint_1"/>-->
-            <joint name="rob1_joint_1"/>
-            <joint name="rob1_joint_2"/>
-            <joint name="rob1_joint_3"/>
-            <joint name="rob1_joint_4"/>
-            <joint name="rob1_joint_5"/>            <joint name="rob1_joint_3" value="0.44897"/>
-            <joint name="rob1_joint_4" value="0.5662"/>
-            <joint name="rob1_joint_5" value="-0.67863"/>
-            <joint name="rob1_joint_6" value="-0.43109"/>
-            <joint name="rob1_joint_6"/>
-        </group>
+        <!--        <group name="extax">-->
+        <!--            <joint name="ext_joint_1"/>-->
+        <!--        </group>-->
         <!--GROUP STATES: Purpose: Define a named state for a particular group, in terms of joint values. This is useful to define states like 'folded arms'-->
         <group_state name="all_zero" group="manipulator">
@@ -37,16 +25,16 @@
             <joint name="rob1_joint_6" value="-0.5671417005127892"/>
         </group_state>
-<!--        <group_state name="zeros" group="extax">-->
-<!--            <joint name="ext_joint_1" value="0"/>-->
-<!--        </group_state>-->
+        <!--        <group_state name="zeros" group="extax">-->
+        <!--            <joint name="ext_joint_1" value="0"/>-->
+        <!--        </group_state>-->
         <!--VIRTUAL JOINT: Purpose: this element defines a virtual joint between a robot link and an external frame of reference (considered fixed with respect to the robot)-->
         <virtual_joint name="world_link" type="fixed" parent_frame="world" child_link="base_link"/>
         <!--DISABLE COLLISIONS: By default it is assumed that any link of the robot could potentially come into collision with any other link in the robot. This tag disables collision checking between a specified pair of links. -->
-<!--        <disable_collisions link1="base_link" link2="extax_link" reason="Adjacent"/>-->
+        <!--        <disable_collisions link1="base_link" link2="extax_link" reason="Adjacent"/>-->
         <disable_collisions link1="base_link" link2="link_1" reason="Adjacent"/>
-<!--        <disable_collisions link1="extax_link" link2="link_1" reason="Never"/>-->
-<!--        <disable_collisions link1="extax_link" link2="link_2" reason="Never"/>-->
+        <!--        <disable_collisions link1="extax_link" link2="link_1" reason="Never"/>-->
+        <!--        <disable_collisions link1="extax_link" link2="link_2" reason="Never"/>-->
         <disable_collisions link1="link_1" link2="link_2" reason="Adjacent"/>
-<!--        <disable_collisions link1="link_1" link2="panels" reason="Never"/>-->
+        <!--        <disable_collisions link1="link_1" link2="panels" reason="Never"/>-->
         <disable_collisions link1="link_1" link2="table" reason="Never"/>
         <disable_collisions link1="link_2" link2="link_3" reason="Adjacent"/>
@@ -60,9 +48,22 @@
         <disable_collisions link1="link_5" link2="toolFrame" reason="Never"/>
         <disable_collisions link1="link_6" link2="toolFrame" reason="Adjacent"/>
-<!--        <disable_collisions link1="base_link" link2="panels" reason="Adjacent"/>-->
+        <!--        <disable_collisions link1="base_link" link2="panels" reason="Adjacent"/>-->
         <disable_collisions link1="base_link" link2="table" reason="Adjacent"/>
-<!--        <disable_collisions link1="extax_link" link2="panels" reason="Never"/>-->
-<!--        <disable_collisions link1="extax_link" link2="table" reason="Default"/>-->
-<!--        <disable_collisions link1="panels" link2="table" reason="Default"/>-->
+        <xacro:property name="use_extax_property" value="${use_extax}"/>
+        <xacro:if value="${use_extax_property == True}">
+            <disable_collisions link1="extax_link" link2="panels" reason="Never"/>
+            <disable_collisions link1="extax_link" link2="table" reason="Default"/>
+            <group name="extax">
+                <joint name="ext_joint_1"/>
+            </group>
+            <group_state name="zeros" group="extax">
+                <joint name="ext_joint_1" value="0"/>
+            </group_state>
+        </xacro:if>
+        <xacro:if value="${use_extax_property == False}">
+            <disable_collisions link1="chuck" link2="table" reason="Default"/>
+            <disable_collisions link1="chuck" link2="base_link" reason="Default"/>
+        </xacro:if>
+        <disable_collisions link1="panels" link2="table" reason="Default"/>
     </xacro:macro>
 </robot>

File: robot_specific_config/abb_irb1200_support/urdf/irb1200.ros2_control.xacro (robot description, xacro)
@@ -19,5 +19,5 @@
                     <!-- The following parameters are used for the MultiMove example only -->
                     <param name="rob1egm_port">6511</param>
-                    <param name="extaxegm_port">6512</param>
+<!--                    <param name="extaxegm_port">6512</param>-->
                 </xacro:unless>
             </hardware>
@@ -88,4 +88,13 @@
                 <state_interface name="velocity"/>
             </joint>
+            <joint name="${prefix}ext_joint_1">
+                <command_interface name="position">
+                </command_interface>
+                <command_interface name="velocity"/>
+                <state_interface name="position">
+                    <param name="initial_value">0.0</param>
+                </state_interface>
+                <state_interface name="velocity"/>
+            </joint>
         </ros2_control>
     </xacro:macro>

File: robot_specific_config/abb_irb1200_support/urdf/irb1200_5_90.xacro (robot description, xacro)
@@ -9,7 +9,9 @@
         <xacro:arg name="robot" default=""/>
         <xacro:property name="robot" value="$(arg robot)"/>
+        <xacro:arg name="use_extax" default="None"/>
+        <xacro:property name="use_extax" value="$(arg use_extax)"/>
 <!--         Robot description-->
         <xacro:include filename="$(find abb_irb1200_support)/urdf/irb1200_5_90_macro.xacro"/>
-        <xacro:abb_irb1200_5_90 prefix="" robot="${robot}"/>
+        <xacro:abb_irb1200_5_90 prefix="" robot="${robot}" use_extax="${use_extax}"/>
 <!--        <xacro:abb_irb1200_5_90 prefix=""/>-->
         <!-- ros2_control -->

File: robot_specific_config/abb_irb1200_support/urdf/irb1200_5_90_macro.xacro (robot description, xacro)
@@ -4,13 +4,14 @@
     <xacro:include filename="$(find optimax_abb_robots)/urdf/ob03_macro.xacro"/>
     <xacro:include filename="$(find optimax_abb_robots)/urdf/ob05_macro.xacro"/>
+    <xacro:include filename="$(find optimax_abb_robots)/urdf/abb_extax.xacro"/>
 <!--    <xacro:macro name="abb_irb1200_5_90" params="prefix">-->
-    <xacro:macro name="abb_irb1200_5_90" params="prefix robot">
+    <xacro:macro name="abb_irb1200_5_90" params="prefix robot use_extax">
         <!-- Check which robot is being used and load in appropriate xacro file -->
         <xacro:property name="robot_property" value="${robot}"/>
         <xacro:if value="${robot_property == 'ob03'}">
-            <xacro:kb06 prefix="${prefix}"/>
+            <xacro:ob03 prefix="${prefix}" use_extax="${use_extax}"/>
         </xacro:if>
         <xacro:if value="${robot_property == 'ob05'}">
-            <xacro:kb04 prefix="${prefix}"/>
+            <xacro:ob05 prefix="${prefix}"/>
         </xacro:if>
         <link name="${prefix}base_link">

Commit message: Seems to be working kind of
The only issue now is the external axis behavior from the joint_traj_compliance_controller or something like that.

File: robot_specific_config/abb_irb1200_5_90_moveit_config/config/abb_irb1200_5_90.srdf.xacro (robot description, xacro)
@@ -1,5 +1,9 @@
 <?xml version="1.0" encoding="utf-8"?>
 <robot xmlns:xacro="http://wiki.ros.org/xacro" name="abb_irb1200_5_90">
+  <xacro:arg name="robot" default=""/>
+  <xacro:property name="robot" value="$(arg robot)"/>
+  <xacro:arg name="use_extax" default=""/>
+  <xacro:property name="use_extax" value="$(arg use_extax)"/>
   <xacro:include filename="$(find abb_irb1200_5_90_moveit_config)/config/abb_irb1200_5_90_macro.srdf.xacro"/>
-  <xacro:abb_irb1200_5_90_srdf/>
+  <xacro:abb_irb1200_5_90_srdf robot="${robot}" use_extax="${use_extax}"/>
 </robot>

File: robot_specific_config/abb_irb1200_5_90_moveit_config/config/abb_irb1200_5_90_macro.srdf.xacro (robot description, xacro)
@@ -1,23 +1,24 @@
 <?xml version="1.0" encoding="utf-8"?>
 <robot xmlns:xacro="http://wiki.ros.org/xacro">
-    <xacro:macro name="abb_irb1200_5_90_srdf">
+    <xacro:include filename="$(find optimax_abb_robots)/srdf/ob03_macro.srdf.xacro"/>
+    <xacro:include filename="$(find optimax_abb_robots)/srdf/ob05_macro.srdf.xacro"/>
+    <xacro:macro name="abb_irb1200_5_90_srdf" params="robot use_extax">
+        <xacro:property name="robot_property" value="${robot}"/>
+        <xacro:property name="use_extax_property" value="${use_extax}"/>
         <group name="manipulator">
             <chain base_link="base_link" tip_link="tool0"/>
         </group>
-<!--        <group name="extax">-->
-<!--            <joint name="ext_joint_1"/>-->
-<!--        </group>-->
-        <group name="whole_station">
-<!--            <joint name="ext_joint_1"/>-->
-            <joint name="rob1_joint_1"/>
-            <joint name="rob1_joint_2"/>
-            <joint name="rob1_joint_3"/>
-            <joint name="rob1_joint_4"/>
-            <joint name="rob1_joint_5"/>            <joint name="rob1_joint_3" value="0.44897"/>
-            <joint name="rob1_joint_4" value="0.5662"/>
-            <joint name="rob1_joint_5" value="-0.67863"/>
-            <joint name="rob1_joint_6" value="-0.43109"/>
-            <joint name="rob1_joint_6"/>
-        </group>
+        <!--        <group name="whole_station">-->
+        <!--&lt;!&ndash;            <joint name="ext_joint_1"/>&ndash;&gt;-->
+        <!--            <joint name="rob1_joint_1"/>-->
+        <!--            <joint name="rob1_joint_2"/>-->
+        <!--            <joint name="rob1_joint_3"/>-->
+        <!--            <joint name="rob1_joint_4"/>-->
+        <!--            <joint name="rob1_joint_5"/>            <joint name="rob1_joint_3" value="0.44897"/>-->
+        <!--            <joint name="rob1_joint_4" value="0.5662"/>-->
+        <!--            <joint name="rob1_joint_5" value="-0.67863"/>-->
+        <!--            <joint name="rob1_joint_6" value="-0.43109"/>-->
+        <!--            <joint name="rob1_joint_6"/>-->
+        <!--        </group>-->
         <!--GROUP STATES: Purpose: Define a named state for a particular group, in terms of joint values. This is useful to define states like 'folded arms'-->
         <group_state name="all_zero" group="manipulator">
@@ -29,24 +30,19 @@
             <joint name="rob1_joint_6" value="-0.009"/>
         </group_state>
-        <group_state name="home" group="manipulator">
-            <joint name="rob1_joint_1" value="0.42577928960737016"/>
-            <joint name="rob1_joint_2" value="0.21565327380088078"/>
-            <joint name="rob1_joint_3" value="0.3686193877257924"/>
-            <joint name="rob1_joint_4" value="0.6880622135409175"/>
-            <joint name="rob1_joint_5" value="-0.7080416122464187"/>
-            <joint name="rob1_joint_6" value="-0.5671417005127892"/>
-        </group_state>
-<!--        <group_state name="zeros" group="extax">-->
-<!--            <joint name="ext_joint_1" value="0"/>-->
-<!--        </group_state>-->
+        <xacro:if value="${robot_property == 'ob03'}">
+            <xacro:ob03_srdf use_extax="${use_extax}"/>
+        </xacro:if>
+        <xacro:if value="${robot_property == 'ob05'}">
+            <xacro:ob05_srdf use_extax="${use_extax}"/>
+        </xacro:if>
         <!--VIRTUAL JOINT: Purpose: this element defines a virtual joint between a robot link and an external frame of reference (considered fixed with respect to the robot)-->
         <virtual_joint name="world_link" type="fixed" parent_frame="world" child_link="base_link"/>
         <!--DISABLE COLLISIONS: By default it is assumed that any link of the robot could potentially come into collision with any other link in the robot. This tag disables collision checking between a specified pair of links. -->
-<!--        <disable_collisions link1="base_link" link2="extax_link" reason="Adjacent"/>-->
+        <!--        <disable_collisions link1="base_link" link2="extax_link" reason="Adjacent"/>-->
         <disable_collisions link1="base_link" link2="link_1" reason="Adjacent"/>
-<!--        <disable_collisions link1="extax_link" link2="link_1" reason="Never"/>-->
-<!--        <disable_collisions link1="extax_link" link2="link_2" reason="Never"/>-->
+        <!--        <disable_collisions link1="extax_link" link2="link_1" reason="Never"/>-->
+        <!--        <disable_collisions link1="extax_link" link2="link_2" reason="Never"/>-->
         <disable_collisions link1="link_1" link2="link_2" reason="Adjacent"/>
-<!--        <disable_collisions link1="link_1" link2="panels" reason="Never"/>-->
+        <!--        <disable_collisions link1="link_1" link2="panels" reason="Never"/>-->
         <disable_collisions link1="link_1" link2="table" reason="Never"/>
         <disable_collisions link1="link_2" link2="link_3" reason="Adjacent"/>
@@ -60,9 +56,20 @@
         <disable_collisions link1="link_5" link2="toolFrame" reason="Never"/>
         <disable_collisions link1="link_6" link2="toolFrame" reason="Adjacent"/>
-<!--        <disable_collisions link1="base_link" link2="panels" reason="Adjacent"/>-->
+        <!--        <disable_collisions link1="base_link" link2="panels" reason="Adjacent"/>-->
         <disable_collisions link1="base_link" link2="table" reason="Adjacent"/>
-<!--        <disable_collisions link1="extax_link" link2="panels" reason="Never"/>-->
-<!--        <disable_collisions link1="extax_link" link2="table" reason="Default"/>-->
-<!--        <disable_collisions link1="panels" link2="table" reason="Default"/>-->
+        <disable_collisions link1="panels" link2="table" reason="Default"/>
+        <xacro:if value="${use_extax_property == True}">
+            <group name="extax">
+                <joint name="ext_joint_1"/>
+            </group>
+            <group_state name="zeros" group="extax">
+                <joint name="ext_joint_1" value="0"/>
+            </group_state>
+            <disable_collisions link1="extax_link" link2="panels" reason="Never"/>
+            <disable_collisions link1="extax_link" link2="table" reason="Default"/>
+        </xacro:if>
+        <xacro:if value="${use_extax_property == False}">
+            <disable_collisions link1="chuck" link2="table" reason="Default"/>
+        </xacro:if>
     </xacro:macro>
 </robot>

File: robot_specific_config/abb_irb1200_support/urdf/irb1200.ros2_control.xacro (robot description, xacro)
@@ -88,4 +88,12 @@
                 <state_interface name="velocity"/>
             </joint>
+            <joint name="${prefix}ext_joint_1">
+                <command_interface name="position"/>
+                <command_interface name="velocity"/>
+                <state_interface name="position">
+                    <param name="initial_value">0.0</param>
+                </state_interface>
+                <state_interface name="velocity"/>
+            </joint>
         </ros2_control>
     </xacro:macro>

File: robot_specific_config/abb_irb1200_support/urdf/irb1200_5_90.xacro (robot description, xacro)
@@ -9,7 +9,9 @@
         <xacro:arg name="robot" default=""/>
         <xacro:property name="robot" value="$(arg robot)"/>
+        <xacro:arg name="use_extax" default=""/>
+        <xacro:property name="use_extax" value="$(arg use_extax)"/>
 <!--         Robot description-->
         <xacro:include filename="$(find abb_irb1200_support)/urdf/irb1200_5_90_macro.xacro"/>
-        <xacro:abb_irb1200_5_90 prefix="" robot="${robot}"/>
+        <xacro:abb_irb1200_5_90 prefix="" robot="${robot}" use_extax="${use_extax}"/>
 <!--        <xacro:abb_irb1200_5_90 prefix=""/>-->
         <!-- ros2_control -->

File: robot_specific_config/abb_irb1200_support/urdf/irb1200_5_90_macro.xacro (robot description, xacro)
@@ -5,12 +5,12 @@
     <xacro:include filename="$(find optimax_abb_robots)/urdf/ob05_macro.xacro"/>
 <!--    <xacro:macro name="abb_irb1200_5_90" params="prefix">-->
-    <xacro:macro name="abb_irb1200_5_90" params="prefix robot">
+    <xacro:macro name="abb_irb1200_5_90" params="prefix robot use_extax">
         <!-- Check which robot is being used and load in appropriate xacro file -->
         <xacro:property name="robot_property" value="${robot}"/>
         <xacro:if value="${robot_property == 'ob03'}">
-            <xacro:kb06 prefix="${prefix}"/>
+            <xacro:ob03 prefix="${prefix}" use_extax="${use_extax}"/>
         </xacro:if>
         <xacro:if value="${robot_property == 'ob05'}">
-            <xacro:kb04 prefix="${prefix}"/>
+            <xacro:ob05 prefix="${prefix}"/>
         </xacro:if>
         <link name="${prefix}base_link">

Commit message: Some changes for running different robots
* abb_irb1200_5_90.srdf.xacro - Added some comments

* abb_irb1200_5_90_macro.srdf.xacro - Removed extax conditional and moved that to a robot specific srdf file.

* irb1200.ros2_control.xacro - Added robot specific control files to be called under specific conditions .

* irb1200_5_90.xacro - Added in a couple parameters to the macro call.

File: robot_specific_config/abb_irb1200_5_90_moveit_config/config/abb_irb1200_5_90.srdf.xacro (robot description, xacro)
@@ -1,8 +1,10 @@
 <?xml version="1.0" encoding="utf-8"?>
 <robot xmlns:xacro="http://wiki.ros.org/xacro" name="abb_irb1200_5_90">
+<!-- Get arguments from launch file -->
   <xacro:arg name="robot" default=""/>
   <xacro:property name="robot" value="$(arg robot)"/>
   <xacro:arg name="use_extax" default=""/>
   <xacro:property name="use_extax" value="$(arg use_extax)"/>
+<!-- Run main srdf macro -->
   <xacro:include filename="$(find abb_irb1200_5_90_moveit_config)/config/abb_irb1200_5_90_macro.srdf.xacro"/>
   <xacro:abb_irb1200_5_90_srdf robot="${robot}" use_extax="${use_extax}"/>

File: robot_specific_config/abb_irb1200_5_90_moveit_config/config/abb_irb1200_5_90_macro.srdf.xacro (robot description, xacro)
@@ -59,17 +59,4 @@
         <disable_collisions link1="base_link" link2="table" reason="Adjacent"/>
         <disable_collisions link1="panels" link2="table" reason="Default"/>
-        <xacro:if value="${use_extax_property == True}">
-            <group name="extax">
-                <joint name="ext_joint_1"/>
-            </group>
-            <group_state name="zeros" group="extax">
-                <joint name="ext_joint_1" value="0"/>
-            </group_state>
-            <disable_collisions link1="extax_link" link2="panels" reason="Never"/>
-            <disable_collisions link1="extax_link" link2="table" reason="Default"/>
-        </xacro:if>
-        <xacro:if value="${use_extax_property == False}">
-            <disable_collisions link1="chuck" link2="table" reason="Default"/>
-        </xacro:if>
     </xacro:macro>
 </robot>

File: robot_specific_config/abb_irb1200_support/urdf/irb1200.ros2_control.xacro (robot description, xacro)
@@ -1,5 +1,8 @@
 <?xml version="1.0"?>
 <robot xmlns:xacro="http://www.ros.org/wiki/xacro">
-    <xacro:macro name="abb_ros2_control" params="name prefix use_fake_hardware:=true rws_ip rws_port">
+    <xacro:include filename="$(find optimax_abb_robots)/urdf/ob03_control_macro.xacro"/>
+    <xacro:macro name="abb_ros2_control" params="name prefix use_fake_hardware:=true rws_ip rws_port use_extax robot">
+        <xacro:property name="use_extax_property" value="${use_extax}"/>
+        <xacro:property name="robot_property" value="${robot}"/>
         <ros2_control name="${name}" type="system">
             <hardware>
@@ -16,8 +19,12 @@
                     <param name="rws_ip">${rws_ip}</param>
                     <!-- The following parameter is used for non-MultiMove only -->
-<!--                    <param name="egm_port">6511</param>-->
+                    <xacro:if value="${use_extax_property == False}">
+                        <param name="egm_port">6511</param>
+                    </xacro:if>
                     <!-- The following parameters are used for the MultiMove example only -->
-                    <param name="rob1egm_port">6511</param>
-                    <param name="extaxegm_port">6512</param>
+                    <xacro:if value="${use_extax_property == True}">
+                        <param name="rob1egm_port">6511</param>
+                        <param name="extaxegm_port">6512</param>
+                    </xacro:if>
                 </xacro:unless>
             </hardware>
@@ -88,12 +95,7 @@
                 <state_interface name="velocity"/>
             </joint>
-            <joint name="${prefix}ext_joint_1">
-                <command_interface name="position"/>
-                <command_interface name="velocity"/>
-                <state_interface name="position">
-                    <param name="initial_value">0.0</param>
-                </state_interface>
-                <state_interface name="velocity"/>
-            </joint>
+            <xacro:if value="${robot_property == 'ob03'}">
+                <xacro:ob03_control prefix="${prefix}"/>
+            </xacro:if>
         </ros2_control>
     </xacro:macro>

File: robot_specific_config/abb_irb1200_support/urdf/irb1200_5_90.xacro (robot description, xacro)
@@ -22,4 +22,6 @@
                 use_fake_hardware="${use_fake_hardware}"
                 rws_ip="${rws_ip}"
-                rws_port="${rws_port}"/>
+                rws_port="${rws_port}"
+                use_extax="${use_extax}"
+                robot="${robot}"/>
     </robot>
